File: KiCAD/AmigaPCI Mainboard-KiCAD REV 70/Agnus-Multi.kicad_sch (KiCad schematic)
At the start: 12 parts, among them J203 RAMEN, J206 CLK/VBB, U202 Agnus_MULTI, U229 74CBT16233

Commit message: AmigaPCI Revision 7.0
Parts:
- added R238: 47R, Resistor_SMD:R_0603_1608Metric, symbol Device:R
- J203: footprint Connector_PinHeader_2.54mm:PinHeader_1x02_P2.54mm_Vertical -> Jumper:SolderJumper-2_P1.3mm_Bridged_RoundedPad1.0x1.5mm
Connections:
- net 7MHz: now also R238.2
- new net ICLK7: R238.1
Other:
- note added: "FUTURE DO NOT POPULATE"
Changed lines of the file:
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@@
 	(title_block
 		(title "AMIGA PCI")
-		(date "2025-07-11")
-		(rev "6.0")
+		(date "2026-04-13")
+		(rev "7.0")
 	)
 	(junction
@@
 	)
 	(junction
+		(at 363.22 31.75)
+		(diameter 0)
+		(color 0 0 0 0)
+	)
+	(junction
 		(at 63.5 232.41)
 		(diameter 0)
@@
 		)
 	)
+	(wire
+		(pts
+			(xy 363.22 36.83) (xy 363.22 31.75)
+		)
+		(stroke
+			(width 0)
+			(type default)
+		)
+	)
 	(bus
 		(pts
@@
 	(wire
 		(pts
-			(xy 294.64 31.75) (xy 372.11 31.75)
+			(xy 294.64 31.75) (xy 363.22 31.75)
 		)
 		(stroke
@@
 		)
 	)
+	(wire
+		(pts
+			(xy 363.22 31.75) (xy 372.11 31.75)
+		)
+		(stroke
+			(width 0)
+			(type default)
+		)
+	)
 	(bus
 		(pts
@@
 	(wire
 		(pts
+			(xy 372.11 36.83) (xy 363.22 36.83)
+		)
+		(stroke
+			(width 0)
+			(type default)
+		)
+	)
+	(wire
+		(pts
 			(xy 387.35 59.69) (xy 387.35 49.53)
 		)
@@
 	(wire
 		(pts
+			(xy 379.73 36.83) (xy 391.16 36.83)
+		)
+		(stroke
+			(width 0)
+			(type default)
+		)
+	)
+	(wire
+		(pts
 			(xy 248.92 118.11) (xy 337.82 118.11)
 		)
@@
 		)
 	)
+	(text "FUTURE DO NOT POPULATE"
+		(exclude_from_sim no)
+		(at 227.584 47.244 0)
+		(effects
+			(font
+				(size 1.27 1.27)
+			)
+		)
+	)
 	(text "SHORT J204 FOR 8372A"
 		(exclude_from_sim no)
@@
 		)
 	)
+	(global_label "ICLK7"
+		(shape output)
+		(at 391.16 36.83 0)
+		(fields_autoplaced yes)
+		(effects
+			(font
+				(size 1.27 1.27)
+			)
+			(justify left)
+		)
+		(property "Intersheetrefs" "${INTERSHEET_REFS}"
+			(at 399.5276 36.83 0)
+			(effects
+				(font
+					(size 1.27 1.27)
+				)
+				(justify left)
+			)
+		)
+	)
 	(global_label "_CDAC"
 		(shape output)
@@
 			)
 		)
-		(property "Footprint" "Connector_PinHeader_2.54mm:PinHeader_1x02_P2.54mm_Vertical"
+		(property "Footprint" "Jumper:SolderJumper-2_P1.3mm_Bridged_RoundedPad1.0x1.5mm"
 			(at 76.2 60.96 0)
 			(effects
@@
 					(unit 1)
 				)
+			)
+		)
+	)
+	(symbol
+		(lib_id "Device:R")
+		(at 375.92 36.83 270)
+		(unit 1)
+		(exclude_from_sim no)
+		(in_bom yes)
+		(on_board yes)
+		(dnp no)
+		(property "Reference" "R238"
+			(at 375.92 34.798 90)
+			(effects
+				(font
+					(size 1.27 1.27)
+				)
+			)
+		)
+		(property "Value" "47R"
+			(at 375.92 37.084 90)
+			(effects
+				(font
+					(size 1.27 1.27)
+				)
+			)
+		)
+		(property "Footprint" "Resistor_SMD:R_0603_1608Metric"
+			(at 375.92 35.052 90)
+			(effects
+				(font
+					(size 1.27 1.27)
+				)
+				(hide yes)
+			)
+		)
+		(property "Datasheet" "~"
+			(at 375.92 36.83 0)
+			(effects
+				(font
+					(size 1.27 1.27)
+				)
+				(hide yes)
+			)
+		)
+		(property "Description" ""
+			(at 375.92 36.83 0)
+			(effects
+				(font
+					(size 1.27 1.27)
+				)
+				(hide yes)
+			)
+		)
+		(pin "1"
+		)
+		(pin "2"
+		)
+		(instances
+			(project "AmigaPCI Mainboard"
+				(path "/72453515-27fe-4336-91f3-e3c8054f7767/2b6a6f7b-f16f-448f-a082-ded618631c29"
+					(reference "R238")
+					(unit 1)
+				)
