File: KiCAD/AmigaPCI Mainboard-KiCAD REV 70/AmigaPCI Mainboard.kicad_sch (KiCad schematic)
At the start: 0 parts

Commit message: AmigaPCI Revision 7.0
Other:
- sheet Clocks and PCI Buffers renamed Clocks, ROM, USB
- sheet MC68040 Level Shift renamed Motorola Bus Logic
- added sheet PCI Bus Logic (pci_bus_logic.kicad_sch)
- sheet Motorola Bus Logic: file mc68040_level_shift.kicad_sch -> motorola_bus_logic.kicad_sch
Changed lines of the file:
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@@
 	(title_block
 		(title "AMIGA PCI")
-		(date "2025-07-11")
-		(rev "6.0")
+		(date "2026-04-13")
+		(rev "7.0")
 	)
 	(text "100 = PCI BUS\n200 = CHIPSET\n300 = VIDEO\n500 = AUDIO\n600 = POWER\n700 = CHIPSET RAM\n800 = VOLTAGE SHIFTER\n900 = ATA"
@@
 	)
 	(sheet
+		(at 76.708 185.166)
+		(size 32.258 11.176)
+		(fields_autoplaced yes)
+		(stroke
+			(width 0.1524)
+			(type solid)
+		)
+		(fill
+			(color 0 0 0 0.0000)
+		)
+		(property "Sheetname" "PCI Bus Logic"
+			(at 76.708 184.4544 0)
+			(effects
+				(font
+					(size 1.27 1.27)
+				)
+				(justify left bottom)
+			)
+		)
+		(property "Sheetfile" "pci_bus_logic.kicad_sch"
+			(at 76.708 196.9266 0)
+			(effects
+				(font
+					(size 1.27 1.27)
+				)
+				(justify left top)
+			)
+		)
+		(instances
+			(project "AmigaPCI Mainboard"
+				(path "/72453515-27fe-4336-91f3-e3c8054f7767"
+					(page "16")
+				)
+			)
+		)
+	)
+	(sheet
 		(at 40.64 100.33)
 		(size 31.75 16.51)
@@
 			(project "AmigaPCI Mainboard"
 				(path "/72453515-27fe-4336-91f3-e3c8054f7767"
-					(page "13")
+					(page "2")
 				)
 			)
@@
 			(project "AmigaPCI Mainboard"
 				(path "/72453515-27fe-4336-91f3-e3c8054f7767"
-					(page "6")
+					(page "5")
 				)
 			)
@@
 			(project "AmigaPCI Mainboard"
 				(path "/72453515-27fe-4336-91f3-e3c8054f7767"
-					(page "8")
+					(page "7")
 				)
 			)
@@
 			(color 0 0 0 0.0000)
 		)
-		(property "Sheetname" "MC68040 Level Shift"
+		(property "Sheetname" "Motorola Bus Logic"
 			(at 40.64 145.3384 0)
 			(effects
@@
 			)
 		)
-		(property "Sheetfile" "mc68040_level_shift.kicad_sch"
+		(property "Sheetfile" "motorola_bus_logic.kicad_sch"
 			(at 40.64 161.7476 0)
 			(effects
@@
 			(project "AmigaPCI Mainboard"
 				(path "/72453515-27fe-4336-91f3-e3c8054f7767"
+					(page "15")
+				)
+			)
+		)
+	)
+	(sheet
+		(at 39.878 29.21)
+		(size 31.75 16.51)
+		(fields_autoplaced yes)
+		(stroke
+			(width 0.1524)
+			(type solid)
+		)
+		(fill
+			(color 0 0 0 0.0000)
+		)
+		(property "Sheetname" "Power and Spares"
+			(at 39.878 28.4984 0)
+			(effects
+				(font
+					(size 1.27 1.27)
+				)
+				(justify left bottom)
+			)
+		)
+		(property "Sheetfile" "power.kicad_sch"
+			(at 39.878 46.2996 0)
+			(effects
+				(font
+					(size 1.27 1.27)
+				)
+				(justify left top)
+			)
+		)
+		(instances
+			(project "AmigaPCI Mainboard"
+				(path "/72453515-27fe-4336-91f3-e3c8054f7767"
 					(page "17")
-				)
-			)
-		)
-	)
-	(sheet
-		(at 40.64 53.34)
-		(size 31.75 16.51)
-		(fields_autoplaced yes)
-		(stroke
-			(width 0.1524)
-			(type solid)
-		)
-		(fill
-			(color 0 0 0 0.0000)
-		)
-		(property "Sheetname" "Power and Spares"
-			(at 40.64 52.6284 0)
-			(effects
-				(font
-					(size 1.27 1.27)
-				)
-				(justify left bottom)
-			)
-		)
-		(property "Sheetfile" "power.kicad_sch"
-			(at 40.64 70.4296 0)
-			(effects
-				(font
-					(size 1.27 1.27)
-				)
-				(justify left top)
-			)
-		)
-		(instances
-			(project "AmigaPCI Mainboard"
-				(path "/72453515-27fe-4336-91f3-e3c8054f7767"
-					(page "3")
 				)
 			)
@@
 			(project "AmigaPCI Mainboard"
 				(path "/72453515-27fe-4336-91f3-e3c8054f7767"
-					(page "15")
+					(page "12")
 				)
 			)
@@
 			(project "AmigaPCI Mainboard"
 				(path "/72453515-27fe-4336-91f3-e3c8054f7767"
-					(page "5")
+					(page "4")
 				)
 			)
@@
 			(project "AmigaPCI Mainboard"
 				(path "/72453515-27fe-4336-91f3-e3c8054f7767"
-					(page "10")
+					(page "9")
 				)
 			)
@@
 			(project "AmigaPCI Mainboard"
 				(path "/72453515-27fe-4336-91f3-e3c8054f7767"
-					(page "11")
+					(page "10")
 				)
 			)
@@
 			(project "AmigaPCI Mainboard"
 				(path "/72453515-27fe-4336-91f3-e3c8054f7767"
-					(page "9")
+					(page "8")
 				)
 			)
@@
 			(project "AmigaPCI Mainboard"
 				(path "/72453515-27fe-4336-91f3-e3c8054f7767"
-					(page "12")
-				)
-			)
-		)
-	)
-	(sheet
-		(at 40.64 29.21)
+					(page "11")
+				)
+			)
+		)
+	)
+	(sheet
+		(at 40.132 53.086)
 		(size 31.75 16.51)
 		(fields_autoplaced yes)
@@
 		)
 		(property "Sheetname" "PCI Bus"
-			(at 40.64 28.4984 0)
+			(at 40.132 52.3744 0)
 			(effects
 				(font
@@
 		)
 		(property "Sheetfile" "pcibus.kicad_sch"
-			(at 40.64 46.9396 0)
-			(effects
-				(font
-					(size 1.27 1.27)
-				)
-				(justify left top)
-			)
-		)
-		(instances
-			(project "AmigaPCI Mainboard"
-				(path "/72453515-27fe-4336-91f3-e3c8054f7767"
-					(page "2")
+			(at 40.132 70.8156 0)
+			(effects
+				(font
+					(size 1.27 1.27)
+				)
+				(justify left top)
+			)
+		)
+		(instances
+			(project "AmigaPCI Mainboard"
+				(path "/72453515-27fe-4336-91f3-e3c8054f7767"
+					(page "13")
 				)
 			)
@@
 			(project "AmigaPCI Mainboard"
 				(path "/72453515-27fe-4336-91f3-e3c8054f7767"
-					(page "16")
+					(page "14")
 				)
 			)
@@
 			(color 0 0 0 0.0000)
 		)
-		(property "Sheetname" "Clocks and PCI Buffers"
+		(property "Sheetname" "Clocks, ROM, USB"
 			(at 76.2 165.6584 0)
 			(effects
@@
 			(project "AmigaPCI Mainboard"
 				(path "/72453515-27fe-4336-91f3-e3c8054f7767"
-					(page "7")
+					(page "6")
 				)
 			)
@@
 			(project "AmigaPCI Mainboard"
 				(path "/72453515-27fe-4336-91f3-e3c8054f7767"
-					(page "14")
-				)
-			)
+					(page "3")
+				)
+			)
