File: KiCAD/AmigaPCI Mainboard-KiCAD REV 70/audio.kicad_sch (KiCad schematic)
At the start: 65 parts, among them CN500 DSP/DVD (RGGL), CN501 AudioJack, Q500 MMBFJ211, Q501 MMBFJ211, Q502 MMBT3906, U220 74LVC08, U500 8364, U501 LF347, U502 LM833

Commit message: AmigaPCI Revision 7.0
Parts:
- added C225: 0.1uF, Capacitor_SMD:C_0603_1608Metric, symbol Device:C_Small
- added R239, R240, R248: 2k7, Resistor_SMD:R_0603_1608Metric, symbol Device:R
- added U208: 74LVC574, Package_SO:TSSOP-20_4.4x6.5mm_P0.65mm, symbol 74xx:74LS574
Connections:
- net GND: now also C225.1, U208.1 (OE), U208.10 (GND)
- net _IPL0: now also U208.12 (Q7); no longer U500.13 (_IPL0)
- net _IPL1: now also U208.13 (Q6); no longer U500.14 (_IPL1)
- net _IPL2: now also U208.14 (Q5); no longer U500.15 (_IPL2)
- new net +3V3: C225.2, R239.1, R240.1, R248.1, U208.20 (VCC)
- new net _CIPL0: R239.2, U208.4 (D2), U500.13 (_IPL0)
- new net _CIPL1: R240.2, U208.3 (D1), U500.14 (_IPL1)
- new net _CIPL2: R248.2, U208.2 (D0), U500.15 (_IPL2)
- new net _CIPLS0: U208.17 (Q2), U208.9 (D7)
- new net _CIPLS1: U208.18 (Q1), U208.8 (D6)
- new net _CIPLS2: U208.19 (Q0), U208.7 (D5)
- new net _CLK40: U208.11 (Cp)
- no-connect marks 0 -> 4
Other:
- note added: "INTERRUPT SYNC"
- moved on the sheet: C506, C507, C508, C509, C510, C511, C522, C523, FB502, R249, R501, R502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
