File: KiCAD/AmigaPCI Mainboard-KiCAD REV 70/audio.kicad_sch (KiCad schematic)
At the start: 70 parts, among them CN500 DSP/DVD (RGGL), CN501 AudioJack, Q500 MMBFJ211, Q501 MMBFJ211, Q502 MMBT3906, U208 74LVC574, U220 74LVC08, U500 8364, U501 LF347, U502 LM833

Commit message: Add JLCPCB part numbers and fix 74LVC244 footprints.
Parts:
- C202, C203, C204, C205, C512, C513: LCSC (none) -> C1622
- C225, C500, C510, C511: LCSC (none) -> C14663
- C501: LCSC (none) -> C59353
- C506, C508, C509: LCSC (none) -> C21120
- C507: LCSC (none) -> C88759
- C514: LCSC (none) -> C57112
- C515, C524: LCSC (none) -> C1631
- C516, C517: LCSC (none) -> C170145
- C518, C519: LCSC (none) -> C1664
- C520, C521: LCSC (none) -> C88755
- C522, C523: LCSC (none) -> C88724
- CN500: LCSC (none) -> C306099
- CN501: LCSC (none) -> C4992459
- FB500, FB501, FB502: LCSC (none) -> C2762183
- Q500, Q501: LCSC (none) -> C3290016
- Q502: LCSC (none) -> C75549
- R239, R240, R248, R512: LCSC (none) -> C13167
- R249, R501, R502, R522, R523, R524, R526: LCSC (none) -> C21190
- R500, R503, R504: LCSC (none) -> C22936
- R505, R507: LCSC (none) -> C23241
- R506: LCSC (none) -> C22765
- R508, R514: LCSC (none) -> C23178
- R509, R510, R511, R513, R515, R516, R517, R525: LCSC (none) -> C25804
- R518, R519: LCSC (none) -> C22940
- R520, R521: LCSC (none) -> C23162
- U208: LCSC (none) -> C7672
- U220: LCSC (none) -> C6053
- U500: LCSC (none) -> C5510465
- U501: LCSC (none) -> C7917
- U502: LCSC (none) -> C127074

Commit message: New hardware rev files.
Gerber
BOM w/JLCPCB part numbers
Pick-n-Place File
Parts:
- R505, R507: LCSC C23241 -> C114635
Changed lines of the file:
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@@
 			)
 		)
-		(property "LCSC" "C23241"
+		(property "LCSC" "C114635"
 			(at 152.4 123.19 0)
 			(effects
@@
 			)
 		)
-		(property "LCSC" "C23241"
+		(property "LCSC" "C114635"
 			(at 152.4 72.39 0)
 			(effects
