File: KiCAD/AmigaPCI Mainboard-KiCAD REV 70/bcontroller.kicad_sch (KiCad schematic)
At the start: 35 parts, among them CN409 SPI, J212 ROM WAIT, U111 74LVC16646, U112 74LVC16646, U409 ICE40HX4K-TQ144, U409F1 W25X20CLSN

Commit message: AmigaPCI Revision 7.0
Parts:
- removed C156, C157, C158, C159: 0.1uF, Capacitor_SMD:C_0603_1608Metric, symbol Device:C_Small
- removed U111, U112: 74LVC16646, Package_SO:SSOP-56_7.5x18.5mm_P0.635mm, symbol AmigaPCI-Symbols:74LVC16646
- added C254: 0.1uF, Capacitor_SMD:C_0603_1608Metric, symbol Device:C_Small
- added J211: FLASH_DIS, Connector_PinHeader_2.54mm:PinHeader_2x01_P2.54mm_Vertical, symbol Connector_Generic:Conn_01x02
- added J409_TP0: U409_TP, Connector_PinHeader_2.54mm:PinHeader_2x01_P2.54mm_Vertical, symbol Connector_Generic:Conn_01x02
- added R270: 22R, Resistor_SMD:R_0603_1608Metric, symbol Device:R
- added R286, R287: 1k, Resistor_SMD:R_0603_1608Metric, symbol Device:R
- added U214: 74LVC244, Package_SO:SSOP-20_4.4x6.5mm_P0.65mm, symbol 74xx:74HCT244
- J900: renamed from JIDE1; value ATA MODES -> AUTOBOOT; footprint Connector_PinHeader_2.54mm:PinHeader_2x03_P2.54mm_Vertical -> Connector_PinHeader_2.54mm:PinHeader_2x01_P2.54mm_Vertical; symbol Connector_Generic:Conn_02x03_Odd_Even -> Connector_Generic:Conn_02x01
Connections:
- net +3V3: now also C254.2, R286.1, R287.1, U214.20 (VCC)
- net GND: now also C254.1, J211.2 (Pin_2), U214.10 (GND), U214.17 (2A0), U214.2 (1A0); no longer J900.3 (Pin_3), J900.5 (Pin_5)
- net U409_SCK: now also U214.12 (1Y3)
- net U409_SDI: now also U214.14 (1Y2)
- net U409_SS: now also U214.18 (1Y0)
- net TP1: now reaches U409.114 (IO0_171)
- net TP1: now also J409_TP0.2 (Pin_2)
- net _AUTOVECTOR: now reaches U409.115 (IO0_172)
- net at U409.125 (IO0_192): now also J211.1 (Pin_1)
- net CLK6: no longer names the net of U409.52 (IO2_82_GBIN4)
- net J901 renamed _LBCEN
- net _LBCEN: no longer J900.4 (Pin_4)
- net J902 renamed TP0
- net TP0: now also J409_TP0.1 (Pin_1); no longer J900.6 (Pin_6)
- net LVCLK7: no longer names the net of U409.49 (IO2_81_GBIN5)
- net PCIAT0: no longer names the net of U409.74 (IO1_110)
- net PCIAT1: no longer names the net of U409.73 (IO1_109)
- net U409_SDO renamed U409_SDOA
- net U409_SDOA: now also U214.4 (1A1)
- net _BPROEN renamed _BRIDGEEN
- net _BREGEN: no longer names the net of U409.91 (IO1_139)
- net _CPUCONF renamed LBC
- net _RSTBTN renamed CDONE
- new net: R270.1, U214.16 (1Y1), U214.5 (2Y1)
- new net SCLKA: U214.11 (2A3), U214.8 (1A3)
- new net SDIA: U214.13 (2A2), U214.6 (1A2)
- new net SDOA: R270.2
- new net U110_SCK: U214.9 (2Y3)
- new net U110_SDI: U214.7 (2Y2)
- new net U110_SDOA: U214.15 (2A1)
- new net U110_SS: U214.3 (2Y0)
- new net _U110EN: R287.2, U214.19 (2OE)
- new net _U409EN: R286.2, U214.1 (1OE)
- no-connect marks 10 -> 8
Other:
- note added: "U409 PROVIDES ADDRESS DECODES, CHIP SELECTS, AND REPLACEMENT GARY FUNCTIONS"
- note removed: "68040 ADDRESS BUS IS LIVE. AD BUS IS LATCHED DURING THE ADDRESS PHASE OF A PCI CYCLE."
- note removed: "PCI ADDRESS LATCH"
- note removed: "U409 PROVIDES ONBOARD DEVICE AUTOCONFIG, ADDRESS DECODE, AND REPLACEMENT GARY FUNCTIONS"
- moved on the sheet: C420, C421, C429, C430, C431, C432, C433, C434, C435, C436, C437, C438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
