File: KiCAD/AmigaPCI Mainboard-KiCAD REV 70/chip_memory.kicad_sch (KiCad schematic)
At the start: 30 parts, among them J1 _CRCS, J3 _CCAS, J4 _CWE, J5 CLKEN, J6 _CRAS, U701 74LVC245, U702 74LVC245, U703 74LVC245, U704 74LVC245, U705 74LVC245, U706 74LVC245, U707 SDRAM(8Mx32)

Commit message: AmigaPCI Revision 7.0
Other:
- note added: "TEST POINTS"
Changed lines of the file:
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@@
 	(title_block
 		(title "AMIGA PCI")
-		(date "2025-08-14")
-		(rev "6.0")
+		(date "2026-04-13")
+		(rev "7.0")
 	)
 	(junction
@@
 		)
 	)
+	(rectangle
+		(start 258.318 194.818)
+		(end 274.828 228.346)
+		(stroke
+			(width 0)
+			(type default)
+		)
+		(fill
+			(type none)
+		)
+	)
+	(text "TEST POINTS"
+		(exclude_from_sim no)
+		(at 266.7 198.12 0)
+		(effects
+			(font
+				(size 1.27 1.27)
+			)
+		)
+	)
