File: KiCAD/AmigaPCI Mainboard-KiCAD REV 70/chip_memory.kicad_sch (KiCad schematic)
At the start: 30 parts, among them J1 _CRCS, J3 _CCAS, J4 _CWE, J5 CLKEN, J6 _CRAS, U701 74LVC245, U702 74LVC245, U703 74LVC245, U704 74LVC245, U705 74LVC245, U706 74LVC245, U707 SDRAM(8Mx32)

Commit message: Add JLCPCB part numbers and fix 74LVC244 footprints.
Parts:
- C701, C702, C703, C704, C705, C706, C707, C708, C709, C710, C711, C712, C713, C714, C715, C716, C717, C718: LCSC (none) -> C14663
- U701, U702, U703, U704, U705, U706: LCSC (none) -> C7848
- U707: LCSC (none) -> C1351836
