File: KiCAD/AmigaPCI Mainboard-KiCAD REV 70/clocks.kicad_sch (KiCad schematic)
At the start: 44 parts, among them U108 74AHC04, U210 AT27C4096, U211 AT27C4096, U219 74AHC04, U223 SST39VF1601C, U812 74LVC245, U813 74LVC245, U814 74LVC245, U815 74LVC08, U816 74LVC245, U817 74LVC245, U818 74LVC245, U819 74LVC245, X1 6MHz, X2 33MHz, X3 28.63636MHz

Commit message: AmigaPCI Revision 7.0
Parts:
- removed C228, C816, C817, C818, C819, C820, C822, C823: 0.1uF, Capacitor_SMD:C_0603_1608Metric, symbol Device:C_Small
- removed R213: 22R, Resistor_SMD:R_0603_1608Metric, symbol Device:R
- removed U812, U813, U814, U816, U817, U818, U819: 74LVC245, Package_SO:TSSOP-20_4.4x6.5mm_P0.65mm, symbol AmigaPCI-Symbols:74LVC245
- removed X1: 6MHz, Oscillator:Oscillator_SMD_ECS_2520MV-xxx-xx-4Pin_2.5x2.0mm, symbol Oscillator:XO32
- added C214, C215, C259: 0.1uF, Capacitor_SMD:C_0603_1608Metric, symbol Device:C_Small
- added C216, C217: 68uF, Capacitor_THT:CP_Radial_D5.0mm_P2.00mm, symbol Device:C_Polarized_Small
- added CN201: USB_A_Stacked, AmigaPCI:USB_A_Wuerth_61400826021_Horizontal_Stacked, symbol Connector:USB_A_Stacked
- added R265: 10k, Resistor_SMD:R_0603_1608Metric, symbol Device:R_Small
- added U225, U226: USBLC6-2SC6, Package_TO_SOT_SMD:SOT-23-6, symbol Power_Protection:USBLC6-2SC6
- added U228: AP2156SG-13, Package_SO:SOIC-8_3.9x4.9mm_P1.27mm, symbol AmigaPCI-Symbols:AP2156SG-13
Connections:
- net GND: now also C214.2, C215.2, C216.2, C217.2, C259.2, CN201.4 (GND1), CN201.8 (GND2), CN201.9 (Shield), R265.2, U225.2 (GND), U226.2 (GND), U228.6 (GND)
- new net +5VSB: C259.1, U228.7 (IN)
- new net USB1+: U225.1 (I/O1)
- new net USB1-: U225.3 (I/O2)
- new net USB1A+: CN201.3 (D1+), U225.6 (I/O1)
- new net USB1A-: CN201.2 (D1-), U225.4 (I/O2)
- new net USB2+: U226.1 (I/O1)
- new net USB2-: U226.3 (I/O2)
- new net USB2A+: CN201.7 (D2+), U226.6 (I/O1)
- new net USB2A-: CN201.6 (D2-), U226.4 (I/O2)
- new net USB5VEN: R265.1, U228.1 (EN1), U228.4 (EN2)
- new net VBUS1: C214.1, C216.1, CN201.1 (VBUS1), U225.5 (VBUS), U228.8 (OUT1)
- new net VBUS2: C215.1, C217.1, CN201.5 (VBUS2), U226.5 (VBUS), U228.5 (OUT2)
- no-connect marks 0 -> 2
Other:
- note added: "CLOCKS, ROM, USB"
- note added: "USB ESD PROTECTION"
- note added: "USB POWER"
- note removed: "AD BUS LEVEL SHIFT"
- note removed: "CLOCKS AND ROMS"
- moved on the sheet: R230
