File: KiCAD/AmigaPCI Mainboard-KiCAD REV 70/cpu.kicad_sch (KiCad schematic)
At the start: 58 parts, among them CN200 DIN41612_03x40, CN712 SPI, U712 ICE40HX4K-TQ144, U712F1 W25X20CLSN, U814 74LVC245, U816 74LVC245, U817 74LVC245

Commit message: AmigaPCI Revision 7.0
Parts:
- removed CN200: DIN41612_03x40, AmigaPCI:DIN41612_C_3x40_Female_Vertical_THT, symbol AmigaPCI-Symbols:DIN41612_03x40
- removed R200: 10k, Resistor_SMD:R_0603_1608Metric, symbol Device:R
- removed R238, R239, R240, R269, R270: 2k7, Resistor_SMD:R_0603_1608Metric, symbol Device:R
- removed RN200, RN201, RN202, RN203, RN204, RN205, RN206, RN207: 2k7, Resistor_THT:R_Array_SIP9, symbol Device:R_Network08
- removed U814, U816, U817: 74LVC245, Package_SO:TSSOP-20_4.4x6.5mm_P0.65mm, symbol AmigaPCI-Symbols:74LVC245
- added C255: 0.1uF, Capacitor_SMD:C_0603_1608Metric, symbol Device:C_Small
- added CN200: DIN41612_03x50, AmigaPCI:DIN41612_C_3x50_Female_Vertical_THT, symbol AmigaPCI-Symbols:DIN41612_03x50
- added J712_TP0: U712_TP, Connector_PinHeader_2.54mm:PinHeader_1x01_P2.54mm_Vertical, symbol Connector_Generic:Conn_01x01
- added R253: 68R, Resistor_SMD:R_0603_1608Metric, symbol Device:R
- added R288, R289: 1k, Resistor_SMD:R_0603_1608Metric, symbol Device:R
- added RN200, RN201, RN202, RN203, RN204, RN205, RN206, RN207, RN209: 3k3, Resistor_SMD:R_Array_Convex_5x0603, symbol AmigaPCI-Symbols:R_SM_Network08
- added U216: 74LVC244, Package_SO:SSOP-20_4.4x6.5mm_P0.65mm, symbol 74xx:74HCT244
- R271: value 2k7 -> 22R
Connections:
- net +1V2: now also CN200.a13 (Pin_a13), CN200.c1 (Pin_c1)
- net +3V3: now also C255.2, CN200.a28 (Pin_a28), CN200.a41 (Pin_a41), CN200.a48 (Pin_a48), CN200.a49 (Pin_a49), CN200.b12 (Pin_b12), CN200.b13 (Pin_b13), CN200.c20 (Pin_c20), CN200.c3 (Pin_c3), CN200.c7 (Pin_c7), R288.1, R289.1, U216.20 (VCC); no longer R242.1
- net +3V3SB: now also CN200.c21 (Pin_c21)
- net +5V: now also R242.1, CN200.a1 (Pin_a1), CN200.a14 (Pin_a14), CN200.a29 (Pin_a29), CN200.a32 (Pin_a32), CN200.a33 (Pin_a33), CN200.a40 (Pin_a40), CN200.a50 (Pin_a50), CN200.c12 (Pin_c12), CN200.c6 (Pin_c6), RN200.5 (common), RN201.5 (common), RN202.5 (common), RN203.5 (common), RN204.5 (common), RN205.10 (common), RN206.5 (common), RN207.5 (common), RN209.5 (common); no longer R271.1
- net A0: now also CN200.b10 (Pin_b10), RN209.3 (R3)
- net A1: now also CN200.a11 (Pin_a11), RN209.4 (R4)
- net A10: now also CN200.b17 (Pin_b17), RN207.6 (R5)
- net A11: now also CN200.a17 (Pin_a17), RN207.7 (R6)
- net A12: now also CN200.a9 (Pin_a9), RN207.8 (R7)
- net A13: now also CN200.b9 (Pin_b9), RN207.9 (R8)
- net A14: now also CN200.a10 (Pin_a10), RN207.1 (R1)
- net A15: now also CN200.c10 (Pin_c10), RN207.2 (R2)
- net A16: now also CN200.c47 (Pin_c47), RN207.3 (R3)
- net A17: now also CN200.b47 (Pin_b47), RN207.4 (R4)
- net A18: now also CN200.a47 (Pin_a47), RN204.7 (R6)
- net A19: now also CN200.c46 (Pin_c46), RN204.6 (R5)
- net A2: now also CN200.b11 (Pin_b11), RN206.6 (R5)
- net A20: now also CN200.b46 (Pin_b46), RN209.1 (R1)
- net A21: now also CN200.c45 (Pin_c45), RN204.4 (R4)
- net A22: now also CN200.a42 (Pin_a42), RN204.3 (R3)
- net A23: now also CN200.a46 (Pin_a46), RN204.1 (R1)
- net A24: now also CN200.a43 (Pin_a43), RN205.1 (R1)
- net A25: now also CN200.b45 (Pin_b45), RN205.6 (R5)
- net A26: now also CN200.b42 (Pin_b42), RN205.2 (R2)
- net A27: now also CN200.c44 (Pin_c44), RN205.7 (R6)
- net A28: now also CN200.c42 (Pin_c42), RN205.3 (R3)
- net A29: now also CN200.c43 (Pin_c43), RN205.4 (R4)
- net A3: now also CN200.c11 (Pin_c11), RN206.7 (R6)
- net A30: now also CN200.b43 (Pin_b43), RN205.8 (R7)
- net A31: now also CN200.b44 (Pin_b44), RN205.9 (R8)
- net A4: now also CN200.a12 (Pin_a12), RN206.8 (R7)
- net A5: now also CN200.b15 (Pin_b15), RN206.9 (R8)
- net A6: now also CN200.a15 (Pin_a15), RN206.1 (R1)
- net A7: now also CN200.b16 (Pin_b16), RN206.2 (R2)
- net A8: now also CN200.a16 (Pin_a16), RN206.3 (R3)
- net A9: now also CN200.c15 (Pin_c15), RN206.4 (R4)
- net CBANK1: now also U712.20 (IO3_13B_GBIN7); no longer U712.49 (IO2_81_GBIN5)
- net CLK40A: now also U712.49 (IO2_81_GBIN5), CN200.a35 (Pin_a35); no longer U712.20 (IO3_13B_GBIN7)
- net D0: now also CN200.a39 (Pin_a39), RN200.6 (R5)
- net D1: now also CN200.c38 (Pin_c38), RN200.7 (R6)
- net D10: now also CN200.c33 (Pin_c33), RN201.8 (R7)
- net D11: now also CN200.b33 (Pin_b33), RN201.9 (R8)
- net D12: now also CN200.c32 (Pin_c32), RN201.1 (R1)
- net D13: now also CN200.c31 (Pin_c31), RN201.2 (R2)
- net D14: now also CN200.c27 (Pin_c27), RN201.3 (R3)
- net D15: now also CN200.b27 (Pin_b27), RN201.4 (R4)
- net D16: now also CN200.b32 (Pin_b32), RN202.9 (R8)
- net D17: now also CN200.a27 (Pin_a27), RN202.8 (R7)
- net D18: now also CN200.b31 (Pin_b31), RN202.7 (R6)
- net D19: now also CN200.b26 (Pin_b26), RN202.6 (R5)
- net D2: now also CN200.a38 (Pin_a38), RN200.8 (R7)
- net D20: now also CN200.a25 (Pin_a25), RN202.4 (R4)
- net D21: now also CN200.c22 (Pin_c22), RN202.3 (R3)
- net D22: now also CN200.b25 (Pin_b25), RN202.2 (R2)
- net D23: now also CN200.c26 (Pin_c26), RN202.1 (R1)
- net D24: now also CN200.b21 (Pin_b21), RN203.9 (R8)
- net D25: now also CN200.a26 (Pin_a26), RN203.8 (R7)
- net D26: now also CN200.a21 (Pin_a21), RN203.7 (R6)
- net D27: now also CN200.b23 (Pin_b23), RN203.6 (R5)
- net D28: now also CN200.b20 (Pin_b20), RN203.4 (R4)
- net D29: now also CN200.a23 (Pin_a23), RN203.3 (R3)
- net D3: now also CN200.b39 (Pin_b39), RN200.9 (R8)
- net D30: now also CN200.b22 (Pin_b22), RN203.2 (R2)
- net D31: now also CN200.a22 (Pin_a22), RN203.1 (R1)
- net D4: now also CN200.b38 (Pin_b38), RN200.1 (R1)
- net D5: now also CN200.c37 (Pin_c37), RN200.2 (R2)
- net D6: now also CN200.b37 (Pin_b37), RN200.3 (R3)
- net D7: now also CN200.c36 (Pin_c36), RN200.4 (R4)
- net D8: now also CN200.a34 (Pin_a34), RN201.6 (R5)
- net D9: now also CN200.b34 (Pin_b34), RN201.7 (R6)
- net GND: now also C255.1, CN200.a2 (Pin_a2), CN200.a31 (Pin_a31), CN200.a36 (Pin_a36), CN200.a37 (Pin_a37), CN200.a44 (Pin_a44), CN200.a45 (Pin_a45), CN200.b14 (Pin_b14), CN200.b6 (Pin_b6), CN200.c16 (Pin_c16), CN200.c17 (Pin_c17), CN200.c24 (Pin_c24), CN200.c25 (Pin_c25), CN200.c4 (Pin_c4), CN200.c49 (Pin_c49), CN200.c50 (Pin_c50), CN200.c8 (Pin_c8), CN200.c9 (Pin_c9), U216.10 (GND), U216.17 (2A0), U216.2 (1A0)
- net PORTSIZE: now also CN200.a8 (Pin_a8)
- net R_W: now also CN200.b19 (Pin_b19)
- net SCL: now also CN200.c40 (Pin_c40)
- net SDA: now also CN200.b41 (Pin_b41)
- net SIZ0: now also CN200.c23 (Pin_c23)
- net SIZ1: now also CN200.a24 (Pin_a24)
- net TM0: now also CN200.a19 (Pin_a19)
- net TM1: now also CN200.c19 (Pin_c19)
- net TM2: now also CN200.a20 (Pin_a20)
- net TT0: now also CN200.c39 (Pin_c39)
- net TT1: now also CN200.b40 (Pin_b40)
- net U712_SCK: now also U216.12 (1Y3)
- net U712_SDI: now also U216.14 (1Y2)
- net U712_SS: now also U216.18 (1Y0)
- net _BB: now also CN200.b8 (Pin_b8)
- net _BG: now also CN200.c29 (Pin_c29)
- net _BR: now also CN200.a18 (Pin_a18)
- net _CPURST: now also CN200.c18 (Pin_c18)
- net _INT2A: now also CN200.c13 (Pin_c13)
- net _INT6: now also CN200.b30 (Pin_b30)
- net _IPL0: now also CN200.c34 (Pin_c34)
- net _IPL1: now also CN200.c35 (Pin_c35)
- net _IPL2: now also CN200.b36 (Pin_b36); no longer R271.2
- net _RESETA: now also CN200.b35 (Pin_b35)
- net _RSTOUT: now also CN200.c41 (Pin_c41)
- net _TACK: now also CN200.b28 (Pin_b28)
- net _TBI: now also CN200.a30 (Pin_a30)
- net _TCI: now also CN200.c30 (Pin_c30)
- net _TEA: now also CN200.c28 (Pin_c28)
- net _TS: now also CN200.b24 (Pin_b24)
- net at U712.37 (IO2_56): now also J712_TP0.1 (Pin_1)
- net LVTT0: no longer names the net of U712.4 (IO3_3B)
- net LVTT0: now also R253.2
- net LVTT1 renamed _DATARDY
- net _DATARDY: now also CN200.b3 (Pin_b3)
- net U712_SDO renamed U712_SDOA
- net U712_SDOA: now also U216.4 (1A1)
- net _LOCK renamed _CPULOCK
- net _CPULOCK: now also CN200.b18 (Pin_b18)
- net _RSTBTN renamed CDONE
- net CDONE: now also CN200.b29 (Pin_b29)
- new net: R271.1, U216.16 (1Y1), U216.5 (2Y1)
- new net LBC: CN200.c14 (Pin_c14)
- new net SCLKA: U216.11 (2A3), U216.8 (1A3)
- new net SCLKB: CN200.a5 (Pin_a5)
- new net SDIA: U216.13 (2A2), U216.6 (1A2)
- new net SDIB: CN200.c5 (Pin_c5)
- new net SDOA: R271.2
- new net SDOB: CN200.b5 (Pin_b5)
- new net U109_SCK: U216.9 (2Y3)
- new net U109_SDI: U216.7 (2Y2)
- new net U109_SDOA: U216.15 (2A1)
- new net U109_SS: U216.3 (2Y0)
- new net _AUTOVECTOR: CN200.b1 (Pin_b1)
- new net _CLK40: R253.1
- new net _LBCEN: CN200.a4 (Pin_a4)
- new net _SPIAEN: CN200.a3 (Pin_a3)
- new net _SPIBEN: CN200.c2 (Pin_c2)
- new net _SPICEN: CN200.b2 (Pin_b2)
- new net _U109EN: R288.2, U216.19 (2OE)
- new net _U712EN: R289.2, U216.1 (1OE)
- no-connect marks 3 -> 27
Other:
- note added: "FPGA PROGRAM"
- note removed: "ADDRESS PHASE DATA PHASE ------------- ------------- PAR _PERR PAR _PERR --------------------------------------- CPU WR BRIDGE PCI BRIDGE PCI CPU RD BRIDGE PCI PCI BRIDGE DMA WR PCI BRIDGE PCI BRIDGE DMA RD PCI BRIDGE BRIDGE PCI"
- note removed: "PCI BUFFERS"
- moved on the sheet: R221, R234, R235, R236, R242, R243, R244, R245, R246, R276, R277, R278
