File: KiCAD/AmigaPCI Mainboard-KiCAD REV 70/floppy.kicad_sch (KiCad schematic)
At the start: 31 parts, among them CN203 DB25_Stack_FemaleAndMale, CN204 INTERNAL FLOPPY, J200 SHORT FOR DF1, J201 1-2 AMIGA DRIVES/2-3 PC DRIVES, J202 1-2 AMIGA DRIVES/2-3 PC DRIVES, J207 TICK, J208 TBASE, U204 8520, U209 74HCT08, U212 74HCT74, U213 74HCT00, U215 74HC03, U219 74AHC04, U305 74HCT08

Commit message: AmigaPCI Revision 7.0
Parts:
- removed RN211: 10k, Resistor_THT:R_Array_SIP9, symbol Device:R_Network08
- removed RN305: 1k, Resistor_THT:R_Array_SIP6, symbol Device:R_Network05
- removed U219: 74AHC04, Package_SO:TSSOP-14_4.4x5mm_P0.65mm, symbol 74xx:74LS04
- added RN211: 10k, Resistor_SMD:R_Array_Convex_5x0603, symbol AmigaPCI-Symbols:R_SM_Network08
- added RN305: 1k, Resistor_SMD:R_Array_Convex_5x0603, symbol AmigaPCI-Symbols:R_SM_Network08
Connections:
- net R_WA is gone; now on net R_W: U204.22 (_W)
- net +5V: now also RN211.10 (common), RN305.10 (common)
- net KBData: now also RN211.3 (R3)
- net PBUSY: now also RN211.9 (R8)
- net PPOUT: now also RN211.8 (R7)
- net PSEL: now also RN211.7 (R6)
- net PSTROBE: now also RN211.2 (R2)
- net _BRST: no longer U204.34 (_RESET)
- net _CHNG: now also RN305.6 (R5)
- net _INDEX: now also RN305.1 (R1)
- net _KBCLK: now also RN211.6 (R5)
- net _PACK: now also RN211.4 (R4)
- net _RDY: now also RN305.2 (R2)
- net _RESETB: now also U204.34 (_RESET)
- net _TRK0: now also RN305.3 (R3)
- net _WPROT: now also RN305.4 (R4)
- no-connect marks 4 -> 9
