File: KiCAD/AmigaPCI Mainboard-KiCAD REV 70/hid.kicad_sch (KiCad schematic)
At the start: 68 parts, among them CN201 USB_A_Stacked, CN202 DB9_Male_Stack, CN206 I2C, CN209 STM DEBUG, CN227 SWD, J209 NRM/PRG, J210 RUN/CAL, U201 74AHCT245, U221 74HCT4066, U222 74HCT4066, U224 74AHCT157, U225 USBLC6-2SC6, U226 USBLC6-2SC6, U227 STM32F205RETx, U228 AP2156SG-13, Y1 8MHz, Y4 32.768KHz

Commit message: AmigaPCI Revision 7.0
Parts:
- removed C214, C215, C259: 0.1uF, Capacitor_SMD:C_0603_1608Metric, symbol Device:C_Small
- removed C216, C217: 68uF, Capacitor_THT:CP_Radial_D5.0mm_P2.00mm, symbol Device:C_Polarized_Small
- removed CN201: USB_A_Stacked, AmigaPCI:USB_A_Wuerth_61400826021_Horizontal_Stacked, symbol Connector:USB_A_Stacked
- removed D204: 1N4148, Diode_SMD:D_SOD-323, symbol Diode:1N4148
- removed R265: 10k, Resistor_SMD:R_0603_1608Metric, symbol Device:R_Small
- removed RN208, RN213: 4k7, Resistor_THT:R_Array_SIP5, symbol Device:R_Network04
- removed U225, U226: USBLC6-2SC6, Package_TO_SOT_SMD:SOT-23-6, symbol Power_Protection:USBLC6-2SC6
- removed U227: STM32F205RETx, Package_QFP:LQFP-64_10x10mm_P0.5mm, symbol MCU_ST_STM32F2:STM32F205RETx
- removed U228: AP2156SG-13, Package_SO:SOIC-8_3.9x4.9mm_P1.27mm, symbol AmigaPCI-Symbols:AP2156SG-13
- added C226, C228: 0.1uF, Capacitor_SMD:C_0603_1608Metric, symbol Device:C_Small
- added CN207: TIMER, Connector_PinHeader_2.54mm:PinHeader_1x04_P2.54mm_Vertical, symbol Connector_Generic:Conn_01x04
- added CN208: UART, Connector_PinHeader_2.54mm:PinHeader_1x03_P2.54mm_Vertical, symbol Connector_Generic:Conn_01x03
- added R269: 220R, Resistor_SMD:R_0603_1608Metric, symbol Device:R_Small
- added R282, R283, R284, R285: 22R, Resistor_SMD:R_0603_1608Metric, symbol Device:R
- added R290, R291, R292: 1k, Resistor_SMD:R_0603_1608Metric, symbol Device:R
- added RN208, RN213: 4k7, Resistor_SMD:R_Array_Convex_5x0603, symbol AmigaPCI-Symbols:R_SM_Network08
- added U227: STM32F205VETx, Package_QFP:LQFP-100_14x14mm_P0.5mm, symbol MCU_ST_STM32F2:STM32F205VETx
- C222: value 7pF -> 4.7pF
- U224: value 74AHCT157 -> 74HCT157; footprint Package_SO:SOIC-16_3.9x9.9mm_P1.27mm -> Package_SO:TSSOP-16_4.4x5mm_P0.65mm
- VC200: value 5-20pF -> 2-5pF; Part Number GKG20015 -> GKG5R015
Connections:
- net +1V2: now also U227.26 (PA3)
- net +3V3: now also R290.1, R291.1, R292.1
- net +3V3SB: now also D203.2 (A), C226.1, C228.1, U227.100 (VDD), U227.11 (VDD), U227.19 (VDD), U227.21 (VREF+), U227.22 (VDDA), U227.28 (VDD), U227.50 (VDD), U227.75 (VDD)
- net +5V: now also RN208.10 (common), RN213.10 (common); no longer D203.2 (A)
- net A2: now also U227.47 (PB10)
- net A3: now also U227.48 (PB11)
- net A4: now also U227.51 (PB12)
- net A5: now also U227.52 (PB13)
- net B0: now also RN208.7 (R6)
- net B1: now also RN213.2 (R2), U227.87 (PD6)
- net BOOT0: now also U227.94 (BOOT0)
- net CLKCAL: now also R269.1, U227.7 (PC13); no longer J210.2 (B)
- net CONS_RX: now also U227.78 (PC10)
- net CONS_TX: now also U227.79 (PC11)
- net DA16: now also U227.90 (PB4)
- net DA17: now also U227.91 (PB5)
- net DA18: now also U227.92 (PB6)
- net DA19: now also U227.93 (PB7)
- net DIO: now also U227.72 (PA13)
- net F1: now also RN213.8 (R7), U227.85 (PD4)
- net FANPWM: now also U227.95 (PB8)
- net FANTACH: now also U227.96 (PB9)
- net FOR0: now also RN208.6 (R5)
- net GND: now also C226.2, C228.2, CN207.2 (Pin_2), CN207.4 (Pin_4), CN208.3 (Pin_3), U227.10 (VSS), U227.20 (VSSA), U227.27 (VSS), U227.74 (VSS)
- net HSCLKIN: now also U227.12 (PH0)
- net HSCLKOUT: now also U227.13 (PH1)
- net KBData: now also U227.65 (PC8)
- net L0: now also RN208.8 (R7)
- net L1: now also RN213.6 (R5), U227.82 (PD1)
- net LSCLKIN: now also U227.8 (PC14)
- net LSCLKOUT: now also U227.9 (PC15)
- net NRST: now also U227.14 (NRST)
- net POWER_LED: now also U227.67 (PA8)
- net POW_SW: now also U227.80 (PC12)
- net PS_ON: now also U227.83 (PD2)
- net PotX0: now also U227.29 (PA4)
- net PotX1: now also U227.81 (PD0)
- net PotY0: now also U227.30 (PA5)
- net PotY1: now also U227.88 (PD7)
- net R0: now also RN208.4 (R4)
- net R1: now also RN213.7 (R6), U227.84 (PD3)
- net SCL: now also U227.69 (PA10)
- net SDA: now also U227.77 (PA15)
- net ST0: now also U227.31 (PA6)
- net ST1: now also U227.32 (PA7)
- net SWCLK: now also U227.76 (PA14)
- net TDO: now also U227.89 (PB3)
- net USB1+: now also U227.71 (PA12)
- net USB1-: now also U227.70 (PA11)
- net USB2+: now also U227.54 (PB15)
- net USB2-: now also U227.53 (PB14)
- net USB5VEN: now also U227.68 (PA9)
- net VBAT_STM: now also U227.6 (VBAT)
- net VMON-12: now also U227.34 (PC5)
- net VMON12: now also U227.33 (PC4)
- net VMON3V3: now also U227.25 (PA2)
- net VMON5: now also U227.23 (PA0)
- net VMON5SB: now also U227.24 (PA1)
- net _FIR0: now also U227.63 (PC6)
- net _FIR1: now also U227.86 (PD5)
- net _HIDEN: now also U227.37 (PB2)
- net _KBCLK: now also U227.66 (PC9)
- net _KBRST: now also U227.64 (PC7)
- net _RTCEN: now also U227.35 (PB0)
- net _STMRST: now also J210.1 (A)
- net at C218.1: now also U227.49 (VCAP_1)
- net at C219.1: now also U227.73 (VCAP_2)
- net R_WA renamed R_W
- net R_W: now also U227.36 (PB1)
- net _Back0 renamed _BACK0
- net _BACK0: now also U227.16 (PC1)
- net _Forward0 renamed _FORWARD0
- net _FORWARD0: now also U227.15 (PC0)
- net _Left0 renamed _LEFT0
- net _LEFT0: now also U227.17 (PC2)
- net _Right0 renamed _RIGHT0
- net _RIGHT0: now also U227.18 (PC3)
- net _STMRSTA: no longer names the net of R224.2
- net _STMRSTA: now also J210.2 (B), R269.2; no longer J210.1 (A)
- new net: R283.2, R285.2, U227.98 (PE1)
- new net: R282.2, R284.2, U227.97 (PE0)
- new net CH1: CN207.1 (Pin_1), U227.59 (PD12)
- new net CH2: CN207.3 (Pin_3), U227.60 (PD13)
- new net RX: CN208.2 (Pin_2), U227.56 (PD9)
- new net SCLKA: R282.1
- new net SCLKB: R284.1
- new net SDIA: R283.1
- new net SDIB: R285.1
- new net SDOA: U227.1 (PE2)
- new net SDOB: U227.43 (PE12)
- new net TX: CN208.1 (Pin_1), U227.55 (PD8)
- new net _SPIAEN: R292.2, U227.46 (PE15)
- new net _SPIBEN: R291.2, U227.45 (PE14)
- new net _SPICEN: R290.2, U227.44 (PE13)
- new net _U109EN: U227.3 (PE4)
- new net _U110EN: U227.2 (PE3)
- new net _U409EN: U227.5 (PE6)
- new net _U712EN: U227.4 (PE5)
- no-connect marks 2 -> 19
Other:
- note removed: "The always on STM can be reset from the +3.3V power domain. When the system is turned off, the STM would interpret this as an asserted reset. We rely on the pullup in the +3.3VSB domain to keep the signal logic high even though the system is shut down. This still allows for a normal reset assertion from the +3.3V domain. The diode isolates the domains."
- note removed: "USB CONNECTOR"
- note removed: "USB ESD PROTECTION"
- note removed: "USB POWER"
- moved on the sheet: BT2, C206, C207, C208, C209, C210, C211, C212, C220, C221, C222, CN206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
