File: KiCAD/AmigaPCI Mainboard-KiCAD REV 70/hid.kicad_sch (KiCad schematic)
At the start: 69 parts, among them CN202 DB9_Male_Stack, CN206 I2C, CN207 TIMER, CN208 UART, CN209 STM DEBUG, CN227 SWD, J209 NRM/PRG, J210 RUN/CAL, U201 74AHCT245, U221 74HCT4066, U222 74HCT4066, U224 74HCT157, U227 STM32F205VETx, Y1 8MHz, Y4 32.768KHz

Commit message: Revision 7.0 Gerbers
Parts:
- U201: value 74AHCT245 -> 74LVC245
Changed lines of the file:
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@@
 	(title_block
 		(title "AMIGA PCI")
-		(date "2026-04-13")
+		(date "2026-04-16")
 		(rev "7.0")
 	)
@@
 			)
 		)
-		(property "Value" "74AHCT245"
+		(property "Value" "74LVC245"
 			(at 59.69 241.808 90)
 			(effects
@@
 			)
 		)
-		(property "Value" "74AHCT245"
+		(property "Value" "74LVC245"
 			(at 146.05 223.52 0)
 			(effects

Commit message: Add JLCPCB part numbers and fix 74LVC244 footprints.
Parts:
- BT2: LCSC (none) -> C238065
- C206, C207, C208, C209, C211, C218, C219, C224, C226, C228, C249, C250, C258, C261: LCSC (none) -> C14663
- C210: LCSC (none) -> C57112
- C212: LCSC (none) -> C15849
- C220, C221: LCSC (none) -> C34243
- C222: LCSC (none) -> C282071
- CN202: LCSC (none) -> C5431655
- CN206, CN207: LCSC (none) -> C124378
- CN208, CN209, J209: LCSC (none) -> C49257
- CN227: LCSC (none) -> C37208
- D202: LCSC (none) -> C460736
- D203: LCSC (none) -> C2286
- F1: LCSC (none) -> C1972812
- J210: LCSC (none) -> C124375
- R201: LCSC (none) -> C23179
- R202, R266: LCSC (none) -> C25804
- R204, R205, R206, R207: LCSC (none) -> C25254
- R224, R255, R256, R257, R258, R259, R262, R263, R264, R268, R290, R291, R292: LCSC (none) -> C21190
- R260, R261: LCSC (none) -> C23186
- R267: LCSC (none) -> C4190
- R269: LCSC (none) -> C22962
- R282, R283, R284, R285: LCSC (none) -> C23345
- RN208, RN213: LCSC (none) -> C728819
- U201: LCSC (none) -> C7848
- U221, U222: LCSC (none) -> C26433
- U224: LCSC (none) -> C2674471
- U227: LCSC (none) -> C81869
- VC200: LCSC (none) -> C3273284
- Y1: LCSC (none) -> C5564812
- Y4: LCSC (none) -> C20340322
