File: KiCAD/AmigaPCI Mainboard-KiCAD REV 70/pci-bridge.kicad_sch (KiCad schematic)
At the start: 44 parts, among them CN109 SPI, CN110 SPI, U109 ICE40HX4K-TQ144, U109F1 W25X20CLSN, U110 ICE40HX4K-TQ144, U110F1 W25X20CLSN

Commit message: AmigaPCI Revision 7.0
Parts:
- removed TP_109: 109_TP, Connector_PinHeader_2.54mm:PinHeader_1x02_P2.54mm_Vertical, symbol Connector_Generic:Conn_01x02
- JATA1: renamed from JPCI1; value PCI MODES -> PIO MODES
Connections:
- net ADLATCH is gone; now on net PCI0: U109.41 (IO2_63)
- net PHASEA_D is gone; now on net _BURST: U109.16 (IO3_10B), U110.81 (IO1_117)
- net _ADEN is gone; now on net _PCIINTEN: U109.22 (IO3_14B)
- net _RSTPCI is gone; now on net _BUSGRANT4: U110.122 (IO0_190)
- net CLK40B: now also U109.49 (IO2_81_GBIN5); no longer U109.52 (IO2_82_GBIN4)
- net CLK40D: now also U110.49 (IO2_81_GBIN5); no longer U110.52 (IO2_82_GBIN4)
- net CLKPCI2: now also U110.129 (IO0_198_GBIN0); no longer U110.93 (IO1_140_GBIN3)
- net IDEDIR: now also U110.84 (IO1_120); no longer U110.83 (IO1_119)
- net IORDY: now also U110.116 (IO0_173); no longer U110.110 (IO0_168)
- net LVAD31: now also U110.91 (IO1_139)
- net PAR_DA: now also U110.83 (IO1_119); no longer U110.82 (IO1_118)
- net PCI0: now also U110.47 (IO2_79); no longer U109.20 (IO3_13B_GBIN7), U110.60 (IO2_95)
- net R_WC: now also U109.17 (IO3_12A), U110.80 (IO1_116); no longer U109.18 (IO3_12B), U110.79 (IO1_115)
- net _BG: now also U110.78 (IO1_114); no longer U109.28 (IO3_23A), U110.76 (IO1_112)
- net _BURST: no longer U109.17 (IO3_12A), U110.80 (IO1_116)
- net _BUSGRANT3: now also U110.124 (IO0_191); no longer U110.125 (IO0_192)
- net _BUSGRANT4: no longer U110.124 (IO0_191)
- net _BUSREQ0: now also U110.110 (IO0_168); no longer U110.112 (IO0_169)
- net _BUSREQ1: now also U110.113 (IO0_170); no longer U110.114 (IO0_171)
- net _BUSREQ2: now also U110.112 (IO0_169); no longer U110.113 (IO0_170)
- net _BUSREQ3: now also U110.115 (IO0_172); no longer U110.116 (IO0_173)
- net _BUSREQ4: now also U110.114 (IO0_171); no longer U110.115 (IO0_172)
- net _CS0A: now also U110.95 (IO1_144); no longer U110.91 (IO1_139)
- net _CS0B: now also U110.85 (IO1_128); no longer U110.84 (IO1_120)
- net _CS1A: now also U110.96 (IO1_146); no longer U110.95 (IO1_144)
- net _CS1B: now also U110.102 (IO1_161); no longer U110.101 (IO1_160)
- net _DIORA: now also U110.97 (IO1_147); no longer U110.96 (IO1_146)
- net _DIORB: now also U110.101 (IO1_160); no longer U110.99 (IO1_152)
- net _DIOWB: now also U110.99 (IO1_152); no longer U110.98 (IO1_148)
- net _IDEHREN: now also U110.90 (IO1_138); no longer U110.88 (IO1_137)
- net _IDEHWEN: now also U110.98 (IO1_148); no longer U110.97 (IO1_147)
- net _IDELATCH: now also U110.87 (IO1_136); no longer U110.85 (IO1_128)
- net _IDELEN: now also U110.88 (IO1_137); no longer U110.87 (IO1_136)
- net _LVCBE0: now also U110.125 (IO0_192); no longer U110.129 (IO0_198_GBIN0)
- net _LVDEVSEL: now also U109.10 (IO3_5B)
- net _LVIRDY: now also U110.139 (IO0_217)
- net _LVPERR: now also U109.37 (IO2_56)
- net _LVSTOP: now also U109.38 (IO2_57); no longer U109.10 (IO3_5B)
- net _LVTS: now also U109.20 (IO3_13B_GBIN7), U109.33 (IO3_25A), U110.21 (IO3_14A_GBIN6); no longer U109.29 (IO3_23B), U110.47 (IO2_79)
- net _PCITIP: now also U109.26 (IO3_18B); no longer U109.25 (IO3_18A)
- net _RESETB: now also U109.25 (IO3_18A), U110.42 (IO2_64); no longer U109.49 (IO2_81_GBIN5), U110.49 (IO2_81_GBIN5)
- net _TACK: now also U109.21 (IO3_14A_GBIN6), U110.93 (IO1_140_GBIN3)
- net _TBI: now also U109.19 (IO3_13A)
- net _PCIEN: now reaches U110.26 (IO3_18B)
- net _PCIEN: now also U109.31 (IO3_24A)
- net LVTT0: now reaches U110.31 (IO3_24A)
- net LVTT1: now reaches U110.32 (IO3_24B)
- net _PCIINTEN: now reaches U110.62 (IO2_102)
- net _PCIBUFEN: now reaches U110.7 (IO3_4A)
- net PPDMA: now reaches U110.8 (IO3_4B)
- net DATADIR: now reaches U110.9 (IO3_5A)
- net _PCIRST: now reaches U109.128 (IO0_197_GBIN1)
- net _CPUBUS: now reaches U109.32 (IO3_24B)
- net _CPUBUS: now also U110.60 (IO2_95)
- net PARITYDIR: now reaches U109.34 (IO3_25B)
- net _BRIDGEEN: now reaches U109.47 (IO2_79)
- net _BRIDGEEN: now also U110.63 (IO2_103_CBSEL0)
- net BUSDIR renamed DMA
- net J100 renamed J901
- net J101 renamed J902
- net J102 renamed J903
- net PCI1 renamed PCIAT2
- net PCIAT2: now also U109.45 (IO2_73); no longer U109.21 (IO3_14A_GBIN6)
- net U109_SDO renamed U109_SDOA
- net U409_CRESET renamed U110_CRESET
- net U409_SCK renamed U110_SCK
- net U409_SDI renamed U110_SDI
- net U409_SDO renamed U110_SDOA
- net U409_SS renamed U110_SS
- removed net _BPROEN: U109.45 (IO2_73), U110.63 (IO2_103_CBSEL0)
- net _BREGEN renamed _WLATCHEN
- net _LVLOCK renamed _LVCPULOCK
- removed net _PCISTART: U109.19 (IO3_13A), U110.78 (IO1_114)
- net _RSTBTN renamed CDONE
- new net LATCHAD: U110.76 (IO1_112)
- new net PCIBUFDIR: U109.28 (IO3_23A)
- new net _ADDRESSEN: U109.52 (IO2_82_GBIN4)
- new net _DATARDY: U109.29 (IO3_23B)
- new net _PCICYCLE: U109.18 (IO3_12B), U110.79 (IO1_115)
- no-connect marks 28 -> 11
