File: KiCAD/AmigaPCI Mainboard-KiCAD REV 70/pci-bridge.kicad_sch (KiCad schematic)
At the start: 43 parts, among them CN109 SPI, CN110 SPI, U109 ICE40HX4K-TQ144, U109F1 W25X20CLSN, U110 ICE40HX4K-TQ144, U110F1 W25X20CLSN

Commit message: Add JLCPCB part numbers and fix 74LVC244 footprints.
Parts:
- C123, C124, C125, C126, C127, C128, C129, C130, C131, C132, C137, C139, C140, C141, C142, C143, C144, C145, C146, C147, C148, C150, C152, C153: LCSC (none) -> C14663
- C136, C138, C149, C151: LCSC (none) -> C96446
- CN109, CN110: LCSC (none) -> C37208
- JATA1: LCSC (none) -> C124384
- R154, R155, R158, R159: LCSC (none) -> C25804
- R156, R157, R160, R161: LCSC (none) -> C22775
- U109, U110: LCSC (none) -> C1521989
- U109F1, U110F1: LCSC (none) -> C34591
