File: KiCAD/AmigaPCI Mainboard-KiCAD REV 70/pcibus.kicad_sch (KiCad schematic)
At the start: 63 parts, among them CN100 PCI32-5V, CN101 PCI32-5V, CN102 PCI32-5V, CN103 PCI32-5V, CN104 PCI32-5V, U815 74LVC08

Commit message: AmigaPCI Revision 7.0
Parts:
- removed RN100: 2k7, Resistor_THT:R_Array_SIP9, symbol Device:R_Network08
- removed RN101: 2k7, Resistor_THT:R_Array_SIP7, symbol Device:R_Network06
- added RN100, RN101: 3k3, Resistor_SMD:R_Array_Convex_5x0603, symbol AmigaPCI-Symbols:R_SM_Network08
Connections:
- net +5V: now also RN100.5 (common), RN101.10 (common)
- net _ACK64: now also RN100.1 (R1)
- net _DEVSEL: now also RN100.6 (R5)
- net _FRAME: now also RN100.9 (R8)
- net _INTA: now also RN101.2 (R2)
- net _INTB: now also RN101.9 (R8)
- net _INTC: now also RN101.1 (R1)
- net _INTD: now also RN101.8 (R7)
- net _IRDY: now also RN100.8 (R7)
- net _LVSYSERR: now also RN101.6 (R5)
- net _PERR: now also RN100.3 (R3)
- net _PLOCK: now also RN101.7 (R6)
- net _REQ64: now also RN100.2 (R2)
- net _STOP: now also RN100.4 (R4)
- net _TRDY: now also RN100.7 (R6)
- net _RSTPCI renamed _PCIRST
- no-connect marks 0 -> 4
Other:
- moved on the sheet: C100, C101, C102, C103, C104, C105, C106, C107, C108, C109, CN100, CN101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
