File: KiCAD/AmigaPCI Mainboard-KiCAD REV 70/pcibus.kicad_sch (KiCad schematic)
At the start: 63 parts, among them CN100 PCI32-5V, CN101 PCI32-5V, CN102 PCI32-5V, CN103 PCI32-5V, CN104 PCI32-5V, U815 74LVC08

Commit message: Add JLCPCB part numbers and fix 74LVC244 footprints.
Parts:
- C100, C101, C102, C103, C104, C105, C106, C107, C108, C109: LCSC (none) -> C57112
- CN100, CN101, CN102, CN103, CN104: LCSC (none) -> C4900616
- R101, R102, R103, R104, R105, R106, R107, R108, R109, R110, R111, R112, R113, R114, R115, R116, R117, R118, R119, R120, R121, R122, R123, R124, R125, R126, R127, R128, R129, R130, R131, R132, R133, R134, R135, R136, R137, R138, R139, R146, R147, R148, R149, R150, R162: LCSC (none) -> C13167
- RN100, RN101: LCSC (none) -> C1731077
- U815: LCSC (none) -> C6053

Commit message: Update PCI Slot Part Number
Parts:
- CN100, CN101, CN102, CN103, CN104: LCSC C4900616 -> C573970
Changed lines of the file:
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@@
 			)
 		)
-		(property "LCSC" "C4900616"
+		(property "LCSC" "C573970"
 			(at 99.06 144.78 0)
 			(effects
@@
 			)
 		)
-		(property "LCSC" "C4900616"
+		(property "LCSC" "C573970"
 			(at 218.44 143.51 0)
 			(effects
@@
 			)
 		)
-		(property "LCSC" "C4900616"
+		(property "LCSC" "C573970"
 			(at 39.37 143.51 0)
 			(effects
@@
 			)
 		)
-		(property "LCSC" "C4900616"
+		(property "LCSC" "C573970"
 			(at 276.86 143.51 0)
 			(effects
@@
 			)
 		)
-		(property "LCSC" "C4900616"
+		(property "LCSC" "C573970"
 			(at 158.75 143.51 0)
 			(effects
