File: KiCAD/AmigaPCI Mainboard-KiCAD REV 70/power.kicad_sch (KiCad schematic)
At the start: 92 parts, among them CN205 Case Fan, CN210 _KBRST, CN601 ATX-24, J11 _REGEN, J2 CLK7, Q202 AO3400A, U200 74LVC2G34, U206 MIC1232, U215 74HC03, U219 74AHC04, U220 74LVC08, U222 74HCT4066, U229 74CBT16233, U231 74LVC08, U232 74AHC1G09, U303 74HCT74, U600 AP2114H-3.3, U601 AP2114H-1.2, U602 LM79L05

Commit message: AmigaPCI Revision 7.0
Parts:
- removed D600, D601, D602, D603: LED, LED_SMD:LED_0603_1608Metric, symbol Device:LED
- removed J2: CLK7, Connector_PinHeader_2.54mm:PinHeader_1x01_P2.54mm_Vertical, symbol Connector_Generic:Conn_01x01
- removed R600: 2k2, Resistor_SMD:R_0603_1608Metric, symbol Device:R_Small
- removed R601, R603: 5k1, Resistor_SMD:R_0805_2012Metric, symbol Device:R_Small
- removed R602: 2k, Resistor_SMD:R_0603_1608Metric, symbol Device:R_Small
- added D204: 1N4148, Diode_SMD:D_SOD-323, symbol Diode:1N4148
- added R250: 1k, Resistor_SMD:R_0603_1608Metric, symbol Device:R
- added unit 6 of U219
- added unit 4 of U219
- CN210: footprint Connector_PinHeader_2.54mm:PinHeader_1x01_P2.54mm_Vertical -> Connector_PinHeader_2.54mm:PinHeader_1x01_P2.54mm_Horizontal
- CN601: footprint Connector_Molex:Molex_Mini-Fit_Jr_5566-24A_2x12_P4.20mm_Vertical -> AmigaPCI:Molex_Mini-Fit_Jr_5566-24A_2x12_P4.20mm_Vertical
- renumbered JCASE1 to CN_CASE1
Connections:
- net +3V3: now also R250.2; no longer C223.1, U200.5 (VCC)
- net +3V3SB: now also C223.1, U200.5 (VCC)
- net GND: no longer U215.1, U215.10, U215.2, U215.9, U219.1
- net _KBRST: now also R250.1
- net _STMRST: now also D204.2 (A); no longer U220.3
- net RESET renamed RESET_BTN
- net _RSTBTN renamed CDONE
- new net: D204.1 (K), U220.3
- no-connect marks 19 -> 28
Other:
- note added: "The always on STM can be reset from the +3.3V power domain. When the system is turned off, the STM would interpret this as an asserted reset. We rely on the pullup in the +3.3VSB domain to keep the signal logic high even though the system is shut down. This still allows for a normal reset assertion from the +3.3V domain. The diode isolates the domains."
- note removed: "CN205"
- note removed: "CN206"
- note removed: "CN207"
- note removed: "CN902"
- note removed: "Just for fun. Omit if desired."
- note removed: "LED Part = LTST-C191KGKT Forward voltage = 2.0v @ 20mA"
- note removed: "POWER RAIL INDICATORS"
- note removed: "R601, R603 = 1/4 WATT"
- moved on the sheet: C201, C223, C251, CN210, U200C, U215C, U220E, U231E, U303B
