File: KiCAD/AmigaPCI Mainboard-KiCAD REV 70/serial.kicad_sch (KiCad schematic)
At the start: 29 parts, among them CN203 DB25_Stack_FemaleAndMale, Q200 MMBT3904, Q201 MMBT3906, U203 8520, U205 AZ75232G, U207 AZ75232G, U209 74HCT08

Commit message: AmigaPCI Revision 7.0
Parts:
- removed R248: 1k, Resistor_SMD:R_0603_1608Metric, symbol Device:R
- added R213: 2k7, Resistor_SMD:R_0603_1608Metric, symbol Device:R
Connections:
- net _INT6: now also R213.2
- net R_WA renamed R_W
- net _BRST renamed _RESETB
- new net +3V3: R213.1
Changed lines of the file:
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@@
 	(title_block
 		(title "AMIGA PCI")
-		(date "2025-07-11")
-		(rev "6.0")
+		(date "2026-04-13")
+		(rev "7.0")
 	)
 	(junction
@@
 	(wire
 		(pts
-			(xy 33.02 142.24) (xy 29.21 142.24)
+			(xy 27.94 142.24) (xy 33.02 142.24)
 		)
 		(stroke
@@
 	(wire
 		(pts
-			(xy 119.38 33.02) (xy 54.61 33.02)
+			(xy 33.02 130.81) (xy 33.02 132.08)
 		)
 		(stroke
@@
 	(wire
 		(pts
-			(xy 99.06 99.06) (xy 106.68 99.06)
+			(xy 119.38 33.02) (xy 54.61 33.02)
 		)
 		(stroke
@@
 	(wire
 		(pts
-			(xy 77.47 162.56) (xy 54.61 162.56)
+			(xy 99.06 99.06) (xy 106.68 99.06)
 		)
 		(stroke
@@
 	(wire
 		(pts
-			(xy 204.47 55.88) (xy 204.47 57.15)
+			(xy 77.47 162.56) (xy 54.61 162.56)
 		)
 		(stroke
@@
 	(wire
 		(pts
-			(xy 308.61 205.74) (xy 339.09 205.74)
+			(xy 204.47 55.88) (xy 204.47 57.15)
 		)
 		(stroke
@@
 	(wire
 		(pts
-			(xy 238.76 41.91) (xy 238.76 73.66)
+			(xy 308.61 205.74) (xy 339.09 205.74)
 		)
 		(stroke
@@
 	(wire
 		(pts
-			(xy 198.12 49.53) (xy 204.47 49.53)
+			(xy 238.76 41.91) (xy 238.76 73.66)
 		)
 		(stroke
@@
 	(wire
 		(pts
-			(xy 77.47 142.24) (xy 33.02 142.24)
+			(xy 198.12 49.53) (xy 204.47 49.53)
 		)
 		(stroke
@@
 	(wire
 		(pts
+			(xy 33.02 142.24) (xy 77.47 142.24)
+		)
+		(stroke
+			(width 0)
+			(type default)
+		)
+	)
+	(wire
+		(pts
 			(xy 111.76 43.18) (xy 111.76 109.22)
 		)
@@
 		)
 	)
+	(wire
+		(pts
+			(xy 33.02 139.7) (xy 33.02 142.24)
+		)
+		(stroke
+			(width 0)
+			(type default)
+		)
+	)
 	(bus
 		(pts
@@
 		)
 	)
-	(global_label "R_WA"
+	(global_label "R_W"
 		(shape input)
 		(at 54.61 127 180)
@@
 		)
 		(property "Intersheetrefs" "${INTERSHEET_REFS}"
-			(at 46.8472 127 0)
+			(at 47.9358 127 0)
 			(effects
 				(font
@@
 		)
 	)
-	(global_label "_BRST"
+	(global_label "_RESETB"
 		(shape input)
 		(at 54.61 162.56 180)
@@
 		)
 		(property "Intersheetrefs" "${INTERSHEET_REFS}"
-			(at 46.0195 162.56 0)
+			(at 43.6421 162.56 0)
 			(effects
 				(font
@@
 	(global_label "_INT6"
 		(shape output)
-		(at 29.21 142.24 180)
+		(at 27.94 142.24 180)
 		(fields_autoplaced yes)
 		(effects
@@
 		)
 		(property "Intersheetrefs" "${INTERSHEET_REFS}"
-			(at 21.1448 142.24 0)
+			(at 19.8748 142.24 0)
 			(effects
 				(font
@@
 	)
 	(symbol
-		(lib_id "Device:R")
-		(at 33.02 138.43 0)
-		(unit 1)
-		(exclude_from_sim no)
-		(in_bom yes)
-		(on_board yes)
-		(dnp no)
-		(property "Reference" "R248"
-			(at 34.798 137.2616 0)
-			(effects
-				(font
-					(size 1.27 1.27)
-				)
-				(justify left)
-			)
-		)
-		(property "Value" "1k"
-			(at 33.02 139.7 90)
-			(effects
-				(font
-					(size 1.27 1.27)
-				)
-				(justify left)
-			)
-		)
-		(property "Footprint" "Resistor_SMD:R_0603_1608Metric"
-			(at 31.242 138.43 90)
-			(effects
-				(font
-					(size 1.27 1.27)
-				)
-				(hide yes)
-			)
-		)
-		(property "Datasheet" "~"
-			(at 33.02 138.43 0)
-			(effects
-				(font
-					(size 1.27 1.27)
-				)
-				(hide yes)
-			)
-		)
-		(property "Description" ""
-			(at 33.02 138.43 0)
-			(effects
-				(font
-					(size 1.27 1.27)
-				)
-				(hide yes)
-			)
-		)
-		(pin "1"
-		)
-		(pin "2"
-		)
-		(instances
-			(project "AmigaPCI Mainboard"
-				(path "/72453515-27fe-4336-91f3-e3c8054f7767/70231775-58c2-469a-996a-fc3c3a4a8de1"
-					(reference "R248")
-					(unit 1)
-				)
-			)
-		)
-	)
-	(symbol
 		(lib_id "AmigaPCI-Symbols:MOS 8520")
 		(at 90.17 243.84 0)
@@
 	)
 	(symbol
-		(lib_name "+5V_1")
-		(lib_id "power:+5V")
-		(at 33.02 134.62 0)
+		(lib_id "power:GND")
+		(at 158.75 125.73 0)
 		(unit 1)
 		(exclude_from_sim no)
@@
 		(on_board yes)
 		(dnp no)
-		(property "Reference" "#PWR0132"
-			(at 33.02 138.43 0)
+		(property "Reference" "#PWR0154"
+			(at 158.75 132.08 0)
 			(effects
 				(font
@@
 			)
 		)
-		(property "Value" "+5V"
-			(at 33.02 130.556 0)
+		(property "Value" "GND"
+			(at 158.877 130.1242 0)
 			(effects
 				(font
@@
 		)
 		(property "Footprint" ""
-			(at 33.02 134.62 0)
+			(at 158.75 125.73 0)
 			(effects
 				(font
@@
 		)
 		(property "Datasheet" ""
-			(at 33.02 134.62 0)
+			(at 158.75 125.73 0)
 			(effects
 				(font
@@
 			)
 		)
-		(property "Description" "Power symbol creates a global label with name \"+5V\""
-			(at 33.02 134.62 0)
+		(property "Description" ""
+			(at 158.75 125.73 0)
 			(effects
 				(font
@@
 			(project "AmigaPCI Mainboard"
 				(path "/72453515-27fe-4336-91f3-e3c8054f7767/70231775-58c2-469a-996a-fc3c3a4a8de1"
-					(reference "#PWR0132")
+					(reference "#PWR0154")
+					(unit 1)
+				)
+			)
+			(project "2000ATX"
+				(path "/bb595301-1c72-49dc-ac6f-007419f3a7fd/00000000-0000-0000-0000-00006065650a"
+					(reference "#PWR0315")
 					(unit 1)
 				)
@@
 	)
 	(symbol
-		(lib_id "power:GND")
-		(at 158.75 125.73 0)
+		(lib_id "power:+3V3")
+		(at 33.02 130.81 0)
 		(unit 1)
 		(exclude_from_sim no)
@@
 		(on_board yes)
 		(dnp no)
-		(property "Reference" "#PWR0154"
-			(at 158.75 132.08 0)
+		(fields_autoplaced yes)
+		(property "Reference" "#PWR282"
+			(at 33.02 134.62 0)
 			(effects
 				(font
@@
 			)
 		)
-		(property "Value" "GND"
-			(at 158.877 130.1242 0)
+		(property "Value" "+3V3"
+			(at 33.02 125.73 0)
 			(effects
 				(font
@@
 		)
 		(property "Footprint" ""
-			(at 158.75 125.73 0)
+			(at 33.02 130.81 0)
 			(effects
 				(font
@@
 		)
 		(property "Datasheet" ""
-			(at 158.75 125.73 0)
+			(at 33.02 130.81 0)
 			(effects
 				(font
@@
 			)
 		)
-		(property "Description" ""
-			(at 158.75 125.73 0)
+		(property "Description" "Power symbol creates a global label with name \"+3V3\""
+			(at 33.02 130.81 0)
 			(effects
 				(font
@@
 		)
 		(instances
-			(project "AmigaPCI Mainboard"
+			(project ""
 				(path "/72453515-27fe-4336-91f3-e3c8054f7767/70231775-58c2-469a-996a-fc3c3a4a8de1"
-					(reference "#PWR0154")
-					(unit 1)
-				)
-			)
-			(project "2000ATX"
-				(path "/bb595301-1c72-49dc-ac6f-007419f3a7fd/00000000-0000-0000-0000-00006065650a"
-					(reference "#PWR0315")
+					(reference "#PWR282")
 					(unit 1)
 				)
@@
 	)
 	(symbol
+		(lib_id "Device:R")
+		(at 33.02 135.89 0)
+		(mirror y)
+		(unit 1)
+		(exclude_from_sim no)
+		(in_bom yes)
+		(on_board yes)
+		(dnp no)
+		(property "Reference" "R213"
+			(at 30.734 138.43 90)
+			(effects
+				(font
+					(size 1.27 1.27)
+				)
+				(justify left)
+			)
+		)
+		(property "Value" "2k7"
+			(at 33.02 137.922 90)
+			(effects
+				(font
+					(size 1.27 1.27)
+				)
+				(justify left)
+			)
+		)
+		(property "Footprint" "Resistor_SMD:R_0603_1608Metric"
+			(at 34.798 135.89 90)
+			(effects
+				(font
+					(size 1.27 1.27)
+				)
+				(hide yes)
+			)
+		)
+		(property "Datasheet" "~"
+			(at 33.02 135.89 0)
+			(effects
+				(font
+					(size 1.27 1.27)
+				)
+				(hide yes)
+			)
+		)
+		(property "Description" ""
+			(at 33.02 135.89 0)
+			(effects
+				(font
+					(size 1.27 1.27)
+				)
+				(hide yes)
+			)
+		)
+		(pin "1"
+		)
+		(pin "2"
+		)
+		(instances
+			(project "AmigaPCI Mainboard"
+				(path "/72453515-27fe-4336-91f3-e3c8054f7767/70231775-58c2-469a-996a-fc3c3a4a8de1"
+					(reference "R213")
+					(unit 1)
+				)
+			)
+		)
+	)
+	(symbol
 		(lib_name "-12V_1")
 		(lib_id "power:-12V")
@@
 			)
 		)
-		(property "Datasheet" " ~"
+		(property "Datasheet" "~"
 			(at 351.79 180.34 0)
 			(effects
