File: KiCAD/AmigaPCI Mainboard-KiCAD REV 70/serial.kicad_sch (KiCad schematic)
At the start: 29 parts, among them CN203 DB25_Stack_FemaleAndMale, Q200 MMBT3904, Q201 MMBT3906, U203 8520, U205 AZ75232G, U207 AZ75232G, U209 74HCT08

Commit message: Add JLCPCB part numbers and fix 74LVC244 footprints.
Parts:
- C227, C230, C231, C232, C233: LCSC (none) -> C14663
- C234, C235, C236: LCSC (none) -> C1588
- C237, C240: LCSC (none) -> C88755
- CN203: LCSC (none) -> C17554757
- D200: LCSC (none) -> C118873
- D201, D400: LCSC (none) -> C460736
- D211: LCSC (none) -> C37574382
- F2: LCSC (none) -> C1972812
- Q200: LCSC (none) -> C84104
- Q201: LCSC (none) -> C75549
- R208, R209: LCSC (none) -> C25804
- R210: LCSC (none) -> C23162
- R211: LCSC (none) -> C25254
- R212: LCSC (none) -> C8218
- R213: LCSC (none) -> C13167
- R214: LCSC (none) -> C21190
- U203: LCSC (none) -> C2332
- U205, U207: LCSC (none) -> C444988
- U209: LCSC (none) -> C131488

Commit message: Updates to revision 7 board.
Change U810 to 74LVC245 buffers
Add CDAC to U712
Add address latch to CIAs
Parts:
- added C242: 0.1uF, Capacitor_SMD:C_0603_1608Metric, symbol Device:C_Small
- added U217: 74HCT273, Package_SO:TSSOP-20_4.4x6.5mm_P0.65mm, symbol 74xx:74LS273
Connections:
- net +5V: now also C242.1, U217.1 (~{Mr}), U217.20 (VCC)
- net A10: now also U217.4 (D1); no longer U203.36 (RS2)
- net A11: now also U217.7 (D2); no longer U203.35 (RS3)
- net A8: now also U217.3 (D0); no longer U203.38 (RS0)
- net A9: now also U217.8 (D3); no longer U203.37 (RS1)
- net GND: now also C242.2, U217.10 (GND)
- net R_W: now also U217.13 (D4); no longer U203.22 (_W)
- new net CIAA10: U203.36 (RS2), U217.5 (Q1)
- new net CIAA11: U203.35 (RS3), U217.2 (Q0)
- new net CIAA8: U203.38 (RS0), U217.9 (Q3)
- new net CIAA9: U203.37 (RS1), U217.6 (Q2)
- new net CIAADL: U217.11 (Cp)
- new net CIAR_W: U203.22 (_W), U217.12 (Q4)
Other:
- note added: "CIA ADDRESS LATCH"
