File: KiCAD/AmigaPCI Mainboard-KiCAD REV 70/video.kicad_sch (KiCad schematic)
At the start: 52 parts, among them CN300 DB15_Female_HighDensity, CN301 Video-Slot, CN302 Video-Slot, J303 HSYNC/COMPSYNC, U300 8362, U301 74AHCT244, U302 74AHCT244, U303 74HCT74, U305 74HCT08

Commit message: AmigaPCI Revision 7.0
Parts:
- removed HY300: VIDIOT, Connector_PinSocket_2.54mm:PinSocket_1x22_P2.54mm_Vertical, symbol AmigaPCI-Symbols:Video Hybrid (VIDIOT)
- removed RN302: 4k7, Resistor_THT:R_Array_SIP5, symbol Device:R_Network04
- added C308, C309, C310, C311, C317: 0.1uF, Capacitor_SMD:C_0603_1608Metric, symbol Device:C_Small
- added Q300, Q301, Q302, Q303, Q304: MMBT3904, Package_TO_SOT_SMD:SOT-23, symbol Transistor_BJT:MMBT3904
- added Q305: MMBT3906, Package_TO_SOT_SMD:SOT-23, symbol Transistor_BJT:MMBT3906
- added R325, R333, R341, R349: 1k, Resistor_SMD:R_0603_1608Metric, symbol Device:R
- added R326, R334, R342: 2k, Resistor_SMD:R_0603_1608Metric, symbol Device:R
- added R327, R335, R343: 3k9, Resistor_SMD:R_0603_1608Metric, symbol Device:R
- added R328, R336, R363: 8k2, Resistor_SMD:R_0603_1608Metric, symbol Device:R
- added R329, R337, R344: 470R, Resistor_SMD:R_0603_1608Metric, symbol Device:R
- added R330, R338, R345: 390R, Resistor_SMD:R_0603_1608Metric, symbol Device:R
- added R331, R332, R339, R340, R346, R347, R352, R362: 75R, Resistor_SMD:R_0603_1608Metric, symbol Device:R
- added R348: 220R, Resistor_SMD:R_0603_1608Metric, symbol Device:R
- added R350: 27k, Resistor_SMD:R_0603_1608Metric, symbol Device:R
- added R351: 150R, Resistor_SMD:R_0603_1608Metric, symbol Device:R
- added R353, R356: 37k4, Resistor_SMD:R_0603_1608Metric, symbol Device:R
- added R354: 13k3, Resistor_SMD:R_0603_1608Metric, symbol Device:R
- added R355: 6k04, Resistor_SMD:R_0603_1608Metric, symbol Device:R
- added R357: 91k, Resistor_SMD:R_0603_1608Metric, symbol Device:R
- added R358: 19k6, Resistor_SMD:R_0603_1608Metric, symbol Device:R
- added R359: 270R, Resistor_SMD:R_0603_1608Metric, symbol Device:R
- added R360: 39R, Resistor_SMD:R_0603_1608Metric, symbol Device:R
- added R361: 36R, Resistor_SMD:R_0603_1608Metric, symbol Device:R
- added RN302: 4k7, Resistor_SMD:R_Array_Convex_5x0603, symbol AmigaPCI-Symbols:R_SM_Network08
- RN301: footprint Resistor_THT:R_Array_SIP9 -> Resistor_SMD:R_Array_Convex_5x0603; symbol Device:R_Network08 -> AmigaPCI-Symbols:R_SM_Network08; Part Number (none) -> YC158TJR-074K7L
Connections:
- net +5V: no longer R308.2
- net +VID: now also RN301.5 (common), C308.2, C309.2, C310.2, C311.2, C317.2, Q300.3 (C), Q301.3 (C), Q302.3 (C), Q303.3 (C), Q305.2 (E), R329.1, R337.1, R344.1, R349.1, R357.1, R359.1, RN302.10 (common); no longer RN301.1 (common)
- net B0: now also R363.1
- net B1: now also U302.3 (2Y0), R343.1; no longer U302.7 (2Y2)
- net B2: now also R342.1
- net B3: now also U302.7 (2Y2), R341.1; no longer U302.3 (2Y0)
- net BLU0: now also RN301.1 (R1); no longer RN301.9 (R8)
- net BLU1: now also RN301.9 (R8), U302.17 (2A0); no longer U302.13 (2A2)
- net BLU2: now also RN301.8 (R7); no longer RN301.4 (R3)
- net BLU3: now also RN301.7 (R6), U302.13 (2A2); no longer U302.17 (2A0)
- net BLUE: now also R347.2
- net COMPVID: now also R362.2
- net G0: now also R336.1
- net G1: now also R335.1
- net G2: now also R334.1
- net G3: now also R333.1
- net GND: now also C308.1, C309.1, C310.1, C311.1, C317.1, R330.2, R331.2, R338.2, R339.2, R345.2, R346.2, R350.2, R351.2, R358.2, R361.2
- net GREEN: now also R340.2
- net GRN0: now also RN301.2 (R2); no longer RN301.8 (R7)
- net GRN1: now also RN301.3 (R3); no longer RN301.7 (R6)
- net GRN2: now also RN301.4 (R4); no longer RN301.6 (R5)
- net GRN3: now also RN301.6 (R5); no longer RN301.5 (R4)
- net R0: now also R328.1
- net R1: now also R327.1
- net R2: now also R326.1
- net R3: now also R325.1
- net RED: now also R332.2
- net RED0: now also RN302.8 (R7)
- net RED1: now also RN302.9 (R8); no longer RN301.3 (R2)
- net RED2: now also RN302.3 (R3)
- net RED3: now also RN302.2 (R2); no longer RN301.2 (R1)
- net SYNC: now also R352.2
- net _COMPSYNC: now also R348.1, R353.1
- new net: Q300.2 (E), R331.1, R332.1
- new net: Q302.1 (B), R341.2, R342.2, R343.2, R344.2, R345.1, R354.1, R363.2
- new net: Q301.1 (B), R333.2, R334.2, R335.2, R336.2, R337.2, R338.1, R356.1
- new net: Q304.3 (C), Q305.1 (B), R359.2
- new net: Q300.1 (B), R325.2, R326.2, R327.2, R328.2, R329.2, R330.1, R355.1
- new net: Q304.1 (B), R353.2, R354.2, R355.2, R356.2, R357.2, R358.1
- new net: Q302.2 (E), R346.1, R347.1
- new net: Q304.2 (E), R360.2, R361.1, R362.1
- new net: Q305.3 (C), R360.1
- new net: Q301.2 (E), R339.1, R340.1
- new net: Q303.2 (E), R351.1, R352.1
- new net: Q303.1 (B), R348.2, R349.2, R350.1
- new net +3V3: R308.2
- no-connect marks 10 -> 16
Other:
- note added: "B&W Composite Optional"
- note added: "VIDEO DAC"
- note removed: "VIDEO HYBRID"
- moved on the sheet: C307, C312, C313, C314, C315, C316, CN300, FB300, FB301, FB302, J303, R226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
