File: KiCAD/AmigaPCI Mainboard-KiCAD REV 70/pci_bus_logic.kicad_sch (KiCad schematic)
At the start: 22 parts, among them U111 74LVC16646, U112 74LVC16646, U800 74LVC2T45, U812 74LVC245, U813 74LVC245, U814 74LVC245, U816 74LVC245, U817 74LVC245, U818 74LVC245, U819 74LVC245

Commit message: Add JLCPCB part numbers and fix 74LVC244 footprints.
Parts:
- C156, C157, C158, C159, C800, C816, C817, C818, C819, C820, C822, C823: LCSC (none) -> C14663
- U111, U112: LCSC (none) -> C2869631
- U800: LCSC (none) -> C15741
- U812, U813, U814, U816, U817, U818, U819: LCSC (none) -> C7848
